File: 221_UnUn.kicad_pcb (KiCad board)
At the start: 2 copper layers, 60.2 x 24.6 mm, 21 parts, among them U1 Core

Commit message: update
Parts:
- removed the REF** at (134.3, 72.4)
- removed the REF** at (134.3, 69.2)
- moved ? 0.79 mm to (112.0, 63.2)
- moved REF** 0.43 mm to (145.9, 63.0)
Changed lines of the file:
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@@
       (drillshape 0)
       (scaleselection 1)
-      (outputdirectory "Gerber/")
+      (outputdirectory "gerber/")
     )
   )
@@
     (pad "1" smd roundrect (at 0 -1.016 270) (size 2 3) (layers "B.Cu" "B.Paste" "B.Mask") (roundrect_rratio 0.25)
       (net 1 "Net-(C1-Pad1)"))
-    (pad "2" thru_hole oval (at -3.8 7.8 270) (size 3 5) (drill 1.5) (layers "*.Cu" "*.Mask")
+    (pad "2" thru_hole oval (at -3.8 7.8 270) (size 3 5) (drill 1.55) (layers "*.Cu" "*.Mask")
       (net 2 "GND"))
-    (pad "2" thru_hole oval (at 3.8 7.8 270) (size 3 5) (drill 1.5) (layers "*.Cu" "*.Mask")
+    (pad "2" thru_hole oval (at 3.8 7.8 270) (size 3 5) (drill 1.55) (layers "*.Cu" "*.Mask")
       (net 2 "GND"))
     (model "${HOMEBREW}/MOLEX_0731713150.wrl"
@@
   )
   (footprint "" (layer "F.Cu")
-    (at 112 63.9572)
+    (at 111.9632 63.1698)
     (fp_text reference "" (at 0 0) (layer "F.SilkS")
         (effects (font (size 1.27 1.27) (thickness 0.15)))
@@
     (pad "3" smd roundrect (at 0 0) (size 2.55 6) (layers "B.Cu" "B.Paste" "B.Mask") (roundrect_rratio 0.09803882353)
       (net 3 "Net-(J2-Pad1)") (pinfunction "x") (pintype "output"))
-  )
-  (footprint "MountingHole:MountingHole_2.1mm" (layer "F.Cu")
-    (at 134.3 69.2)
-    (descr "Mounting Hole 2.1mm, no annular")
-    (tags "mounting hole 2.1mm no annular")
-    (attr exclude_from_pos_files exclude_from_bom)
-    (fp_text reference "REF**" (at 0 -3.2) (layer "F.SilkS") hide
-        (effects (font (size 1 1) (thickness 0.15)))
-    )
-    (fp_text value "MountingHole_2.1mm" (at 0 3.2) (layer "F.Fab") hide
-        (effects (font (size 1 1) (thickness 0.15)))
-    )
-    (fp_text user "${REFERENCE}" (at 0 0) (layer "F.Fab") hide
-        (effects (font (size 1 1) (thickness 0.15)))
-    )
-    (fp_circle (center 0 0) (end 2.1 0)
-      (stroke (width 0.15) (type solid)) (fill none) (layer "Cmts.User"))
-    (fp_circle (center 0 0) (end 2.35 0)
-      (stroke (width 0.05) (type solid)) (fill none) (layer "F.CrtYd"))
-    (pad "" np_thru_hole circle (at 0 0) (size 1.5 1.5) (drill 1.5) (layers "F&B.Cu" "*.Mask"))
   )
   (footprint "Symbol:OSHW-Symbol_6.7x6mm_SilkScreen" (layer "F.Cu")
@@
   )
   (footprint "MountingHole:MountingHole_6.4mm_M6" (layer "F.Cu")
-    (at 146.3802 63.0428)
+    (at 145.9484 62.992)
     (descr "Mounting Hole 6.4mm, no annular, M6")
     (tags "mounting hole 6.4mm no annular m6")
@@
     (fp_circle (center 0 0) (end 2.35 0)
       (stroke (width 0.05) (type solid)) (fill none) (layer "F.CrtYd"))
-    (pad "" np_thru_hole circle (at 0 0) (size 2.1 2.1) (drill 2.5) (layers "F&B.Cu" "*.Mask"))
+    (pad "" np_thru_hole circle (at 0 0) (size 2.5 2.5) (drill 2.5) (layers "F&B.Cu" "*.Mask"))
   )
   (footprint "MountingHole:MountingHole_2.1mm" (layer "F.Cu")
@@
     (fp_circle (center 0 0) (end 2.35 0)
       (stroke (width 0.05) (type solid)) (fill none) (layer "F.CrtYd"))
-    (pad "" np_thru_hole circle (at 0 0) (size 2.1 2.1) (drill 2.5) (layers "F&B.Cu" "*.Mask"))
+    (pad "" np_thru_hole circle (at 0 0) (size 2.5 2.5) (drill 2.5) (layers "F&B.Cu" "*.Mask"))
   )
   (footprint "MountingHole:MountingHole_2.1mm" (layer "F.Cu")
@@
   )
   (footprint "MountingHole:MountingHole_2.1mm" (layer "F.Cu")
-    (at 134.3 72.39)
-    (descr "Mounting Hole 2.1mm, no annular")
-    (tags "mounting hole 2.1mm no annular")
-    (attr exclude_from_pos_files exclude_from_bom)
-    (fp_text reference "REF**" (at 0 -3.2) (layer "F.SilkS") hide
-        (effects (font (size 1 1) (thickness 0.15)))
-    )
-    (fp_text value "MountingHole_2.1mm" (at 0 3.2) (layer "F.Fab") hide
-        (effects (font (size 1 1) (thickness 0.15)))
-    )
-    (fp_text user "${REFERENCE}" (at 0 0) (layer "F.Fab") hide
-        (effects (font (size 1 1) (thickness 0.15)))
-    )
-    (fp_circle (center 0 0) (end 2.1 0)
-      (stroke (width 0.15) (type solid)) (fill none) (layer "Cmts.User"))
-    (fp_circle (center 0 0) (end 2.35 0)
-      (stroke (width 0.05) (type solid)) (fill none) (layer "F.CrtYd"))
-    (pad "" np_thru_hole circle (at 0 0) (size 1.5 1.5) (drill 1.5) (layers "F&B.Cu" "*.Mask"))
-  )
-  (footprint "MountingHole:MountingHole_2.1mm" (layer "F.Cu")
     (at 139.4 72.39)
     (descr "Mounting Hole 2.1mm, no annular")
@@
     (fp_circle (center 0 0) (end 2.35 0)
       (stroke (width 0.05) (type solid)) (fill none) (layer "F.CrtYd"))
-    (pad "" np_thru_hole circle (at 0 0) (size 2.1 2.1) (drill 2.5) (layers "F&B.Cu" "*.Mask"))
+    (pad "" np_thru_hole circle (at 0 0) (size 2.5 2.5) (drill 2.5) (layers "F&B.Cu" "*.Mask"))
   )
   (footprint "Capacitor_SMD:C_1206_3216Metric_Pad1.33x1.80mm_HandSolder" (layer "B.Cu")
@@
   (gr_line (start 137.280627 80.592109) (end 150.834956 80.599915)
     (stroke (width 0.1) (type default)) (layer "Edge.Cuts"))
-  (gr_text "DG1JAN" (at 142.24 59.944 230) (layer "F.SilkS")
-    (effects (font (size 1.2 1.3) (thickness 0.3)) (justify left bottom))
-  )
-  (gr_text "(CC BY-SA 4.0)" (at 110.5408 65.8368 180) (layer "F.SilkS")
+  (gr_text "DG1JAN" (at 133.1468 70.8914 270) (layer "F.SilkS")
+    (effects (font (size 1.5 1.2) (thickness 0.2) bold))
+  )
+  (gr_text "221-UnUn" (at 143.891 74.9554 180) (layer "F.SilkS")
+    (effects (font (size 1.5 1.5) (thickness 0.3) bold))
+  )
+  (gr_text "(CC BY-SA 4.0)" (at 110.5154 65.786 180) (layer "F.SilkS")
     (effects (font (size 1 1) (thickness 0.2) bold))
   )
-  (gr_text "221-UnUn" (at 149.987 74.168 180) (layer "F.SilkS")
-    (effects (font (size 1.2 1.5) (thickness 0.3)) (justify left bottom))
-  )
   (segment (start 106.3975 71.8915) (end 105.166 70.66) (width 1.3) (layer "B.Cu") (net 1))
